File: Glider.brd (EAGLE design)
At the start: 69.1 x 53.3 mm, 49 parts, among them IC1 LD6806, IC2 LM555D, IC3 4050D, IC4 DS1307SO8, IC5 BMP180, IC6 LSM9DS0, Q1 32.768Khz, Q4 MOSFET-NCHANNELBSS123LT1G, Q5 MOSFET-NCHANNELBSS123LT1G

Commit message: Didn't save...
Routing:
- net +5V: track 128.8 -> 135.2 mm
- net GND: vias 19 -> 20
Changed lines of the file:
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@@
 <layer number="20" name="Dimension" color="15" fill="1" visible="yes" active="yes"/>
 <layer number="21" name="tPlace" color="7" fill="1" visible="yes" active="yes"/>
-<layer number="22" name="bPlace" color="7" fill="1" visible="yes" active="yes"/>
+<layer number="22" name="bPlace" color="7" fill="1" visible="no" active="yes"/>
 <layer number="23" name="tOrigins" color="15" fill="1" visible="yes" active="yes"/>
-<layer number="24" name="bOrigins" color="15" fill="1" visible="yes" active="yes"/>
+<layer number="24" name="bOrigins" color="15" fill="1" visible="no" active="yes"/>
 <layer number="25" name="tNames" color="7" fill="1" visible="yes" active="yes"/>
 <layer number="26" name="bNames" color="7" fill="1" visible="no" active="yes"/>
@@
 <layer number="42" name="bRestrict" color="1" fill="10" visible="no" active="yes"/>
 <layer number="43" name="vRestrict" color="2" fill="10" visible="no" active="yes"/>
-<layer number="44" name="Drills" color="7" fill="1" visible="no" active="yes"/>
+<layer number="44" name="Drills" color="7" fill="1" visible="yes" active="yes"/>
 <layer number="45" name="Holes" color="7" fill="1" visible="yes" active="yes"/>
 <layer number="46" name="Milling" color="3" fill="1" visible="no" active="yes"/>
@@
 <wire x1="69.1359" y1="5.0921" x2="69.1359" y2="5.0997" width="0" layer="20"/>
 <circle x="65.5421" y="44.4551" radius="0.8519" width="0.3048" layer="21"/>
-<text x="29.21" y="43.18" size="1.27" layer="25">HAAG
-Duke Robotics 2014</text>
 <wire x1="69.215" y1="6.985" x2="58.42" y2="6.985" width="0.6096" layer="41"/>
 <wire x1="58.42" y1="6.985" x2="58.42" y2="19.05" width="0.6096" layer="41"/>
@@
 <wire x1="3.81" y1="19.685" x2="5.08" y2="20.955" width="0.3048" layer="25"/>
 <wire x1="3.81" y1="20.955" x2="5.08" y2="19.685" width="0.3048" layer="25"/>
-<text x="56.515" y="40.64" size="1.27" layer="21">R-
+<text x="66.675" y="15.875" size="1.27" layer="21">R-
 R+
 F-
@@
 B+</text>
 <rectangle x1="43.815" y1="8.255" x2="45.085" y2="9.525" layer="21"/>
+<text x="37.465" y="41.275" size="1.27" layer="25" font="vector" ratio="24" align="center">HAAG
+Duke Robotics
+2014</text>
 </plain>
 <attributes>
@@
 <contactref element="C8" pad="1"/>
 <contactref element="IC1" pad="3"/>
-<wire x1="40.64" y1="5.5" x2="40.64" y2="6.35" width="0" layer="19" extent="1-16"/>
 <wire x1="25.67" y1="28.645" x2="25.67" y2="29.48" width="0.4064" layer="1"/>
 <wire x1="25.67" y1="29.48" x2="26.035" y2="29.845" width="0.4064" layer="1"/>
@@
 <wire x1="38.1" y1="5.485" x2="40.625" y2="5.485" width="0.3048" layer="1"/>
 <wire x1="40.625" y1="5.485" x2="40.64" y2="5.5" width="0.3048" layer="1"/>
-<wire x1="38.608" y1="5.08" x2="38.1" y2="5.485" width="0" layer="19" extent="1-16"/>
+<wire x1="38.1" y1="5.485" x2="40.64" y2="5.485" width="0.3048" layer="1"/>
+<wire x1="40.64" y1="5.485" x2="40.64" y2="5.08" width="0.3048" layer="1"/>
+<wire x1="38.1" y1="5.485" x2="38.608" y2="5.485" width="0.6096" layer="1"/>
+<wire x1="38.608" y1="5.485" x2="38.608" y2="2.54" width="0.6096" layer="1"/>
 </signal>
 <signal name="GND">
@@
 <via x="35.56" y="33.02" extent="1-16" drill="0.3302" diameter="0.508"/>
 <via x="31.75" y="36.83" extent="1-16" drill="0.3302" diameter="0.508"/>
-<via x="36.83" y="39.37" extent="1-16" drill="0.3302" diameter="0.508"/>
+<via x="41.275" y="38.1" extent="1-16" drill="0.3302" diameter="0.508"/>
 <via x="39.37" y="45.085" extent="1-16" drill="0.3302" diameter="0.508"/>
 <via x="7.62" y="34.29" extent="1-16" drill="0.3302" diameter="0.508"/>
@@
 <via x="30.48" y="5.715" extent="1-16" drill="0.3302" diameter="0.508"/>
 <via x="11.43" y="43.815" extent="1-16" drill="0.3302" diameter="0.508"/>
+<via x="66.04" y="5.08" extent="1-16" drill="0.3302" diameter="0.508"/>
 </signal>
 <signal name="RESET">

Commit message: Final check, added BOM as .csv
Parts:
- removed LED4: red, adafruit:CHIPLED_0805
- added LED1: (no value), led:CHIPLED_0805
- C14, C15: value (none) -> 47u
- IC1: value LD6806 -> (none); device AWJLEagleLib:SOT-753 -> AWJLEagleLib:SOT-23
- R6: value (none) -> 1k
- moved R6 6.35 mm to (29.2, 45.1)
- moved LED3 2.54 mm to (27.3, 45.1)
- moved C8 1.27 mm to (39.4, 31.1)
- moved R3 1.27 mm to (41.9, 31.1)
- moved C3 1.27 mm to (21.6, 45.1)
- turned IC1 to 180 degrees
Connections:
- net +3V3: now also IC1.2; no longer IC1.5
- net +5V: no longer IC1.1
- net GND: now also IC1.1, LED1.C; no longer IC1.2, LED4.C
- net N$6: now also LED1.A; no longer LED4.A
Routing:
- net +5V: track 135.2 -> 129.3 mm
- net SCK: track 20.1 -> 23.4 mm, vias 2 -> 1
- net N$12: track 11.5 -> 12.2 mm
- net MISO: track 28.6 -> 29.2 mm
