File: Glider.sch (EAGLE design)
At the start: 37 parts, among them IC1 MCP1700-330, IC2 LM555D, IC3 4050D, Q1 32.768Khz

Commit message: First draft of control board
Parts:
- removed I2C: rtc pins, pinhead:PINHD-1X2
- removed JP1: sd pins, pinhead:PINHD-1X4
- removed JP11: led pins, pinhead:PINHD-1X2
- removed JP12: 3v jumper, jumper:JP1E
- removed JP14: (no value), pinhead:PINHD-1X4
- removed JP2: d8-aref, adafruit:PINHD-1X8BIG
- removed JP4: D0-D7, adafruit:PINHD-1X8BIG
- removed JP7, JP9: (no value), adafruit:PINHD-1X6B
- removed LED1: red, adafruit:LEDCHIPLED_0805
- removed LED2: green, adafruit:LEDCHIPLED_0805
- removed R8, R9: (no value), rcl:R-US_R0805
- added C6: 15u, rcl:C-USC0805
- added C8: 0.1uF, adafruit:C-USC0805
- added D1: BAS40-04, diode:BAS40-04
- added Q2, Q3: (no value), HAAG:NTD20N06LT4G
- added X1: (no value), con-wago-508:W237-06P
- C5: value (none) -> 10n; device rcl:C-EUC0805 -> rcl:C-USC0805
- IC1: value MCP1700-330 -> LD6806; device adafruit:MCP1700TRI -> AWJLEagleLib:LD6806
- R3: value 1k -> 10k; device adafruit:R-US_R0805 -> rcl:R-EU_R0805
- R4: value 1k -> 100k; device adafruit:R-US_R0805 -> rcl:R-TRIMM3214W
- renumbered U$2 to IC4, U$3 to SD
Connections:
- removed net 3.3V: JP12.2, JP7.5, U$1.3V
- removed net N$101: JP4.8, U$1.D7
- removed net N$111: JP2.8, U$1.D8
- removed net N$14: LED1.A, R3.1
- removed net N$15: JP7.1, U$1.VIN
- removed net N$154: JP9.1, U$1.A0
- removed net N$164: JP9.2, U$1.A1
- removed net N$17: JP11.2, R3.2
- removed net N$18: LED2.A, R4.2
- removed net N$181: JP9.3, U$1.A2
- removed net N$182: JP9.4, U$1.A3
- removed net N$20: JP11.1, R4.1
- removed net N$87: JP4.1, U$1.D0
- removed net N$88: JP4.2, U$1.D1
- removed net N$89: JP4.3, U$1.D2
- removed net N$90: JP4.4, U$1.D3
- removed net N$98: JP4.5, U$1.D4
- removed net N$99: JP4.6, U$1.D5
- removed net RTC_SCL: I2C.1, IC4.SCL, JP9.6, R1.2, U$1.A5
- removed net RTC_SDA: I2C.2, IC4.SDA, JP9.5, R2.2, U$1.A4
- removed net SD_CD: JP14.1, SD.CARD_DETECT
- removed net SD_WP: JP14.2
- removed net VDD: SD.VDD
- new net FLASH: Q2.D, X1-4.KL
- new net I2C_SCL: IC4.SCL, R1.2, SENSOR.3, U$1.A5
- new net I2C_SDA: IC4.SDA, R2.2, SENSOR.4, U$1.A4
- new net N$10: C5.1, IC2.CV
- new net N$12: IC2.DIS, Q2.G, R3.1
- new net N$7: D1.A1, R4.A
- new net N$8: D1.C2, R4.E
- new net N$9: C6.1, D1.C1A2, IC2.THR, IC2.TR
- new net RELEASE: Q3.D, X1-6.KL
- new net V+: X1-1.KL, X1-3.KL, X1-5.KL
- net +3V3: now also SD.VDD; no longer JP12.1, JP14.4
- net +5V: now also C8.1, IC1.EN, IC2.R, R3.2, SENSOR.5, SENSOR.6; no longer JP7.4
- net GND: now also C5.2, C6.2, C8.2, IC3D.I, IC3E.I, IC3F.I, Q2.S, Q3.S, SD.GND1, SENSOR.1, SENSOR.2, X1-2.KL; no longer JP2.2, JP7.2, JP7.3, LED1.C, LED2.C, SD.CARD_DETECT1
- net MISO: no longer JP1.1, JP2.4
- net MOSI: now also IC3B.I; no longer IC3A.I, JP1.2, JP2.5
- net N$100: now also Q3.G; no longer JP4.7
- net N$108: no longer JP2.1
- net N$110: no longer JP2.7
- net N$5: now also IC2.Q, R4.S; no longer IC3D.I, R5.2
- net RESET: no longer JP7.6
- net SCK: now also IC3A.I; no longer IC3C.I, JP1.4, JP2.3
- net SD_CS: now also IC3C.I, R5.2; no longer JP1.3, JP2.6
- net SD_CSIN: now also IC3C.O; no longer IC3D.O
- net SD_DATAIN: now also IC3B.O; no longer IC3A.O
- net SD_SCKIN: now also IC3A.O; no longer IC3C.O
- net SQW: no longer JP14.3
Other:
- note added: "f = 1.44 / (R4*C6)"
- moved on the sheet: C1, C2, C3, C4, C5, IC2, IC3A, IC3B, IC3C, IC3D, IC3P, LED4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

Commit message: First draft layout - to check!
Parts:
- added C7: 0.1uF, adafruit:C-USC0805
- added R8: 10k, rcl:R-EU_R0805
Connections:
- net +5V: now also C7.1
- net GND: now also C7.2, R8.1
- net N$100: now also R8.2
Changed lines of the file:
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@@
 <part name="P+7" library="supply1" deviceset="+5V" device=""/>
 <part name="GND15" library="supply1" deviceset="GND" device=""/>
+<part name="C7" library="adafruit" deviceset="C-US" device="C0805" value="0.1uF"/>
+<part name="R8" library="rcl" deviceset="R-EU_" device="R0805" value="10k"/>
 </parts>
 <sheets>
@@
 <instance part="P+5" gate="1" x="96.52" y="160.02"/>
 <instance part="U$1" gate="G$1" x="45.72" y="96.52"/>
-<instance part="GND7" gate="1" x="40.64" y="139.7" rot="MR180"/>
+<instance part="GND7" gate="1" x="38.1" y="139.7" rot="MR180"/>
 <instance part="+3V8" gate="G$1" x="111.76" y="40.64"/>
 <instance part="IC3" gate="B" x="167.64" y="99.06" rot="R180"/>
@@
 <attribute name="VALUE" x="138.938" y="212.2424" size="1.778" layer="96" rot="R180"/>
 </instance>
-<instance part="GND14" gate="1" x="106.68" y="114.3" rot="MR0"/>
+<instance part="GND14" gate="1" x="106.68" y="109.22" rot="MR0"/>
 <instance part="P+7" gate="1" x="157.48" y="157.48"/>
 <instance part="GND15" gate="1" x="157.48" y="132.08" rot="MR0"/>
+<instance part="C7" gate="G$1" x="48.26" y="20.32"/>
+<instance part="R8" gate="G$1" x="88.9" y="121.92" rot="R90"/>
 </instances>
 <busses>
@@
 <junction x="25.4" y="25.4"/>
 <pinref part="IC1" gate="G$1" pin="IN"/>
-<wire x1="40.64" y1="25.4" x2="55.88" y2="25.4" width="0.1524" layer="91"/>
+<wire x1="40.64" y1="25.4" x2="48.26" y2="25.4" width="0.1524" layer="91"/>
 <pinref part="C8" gate="G$1" pin="1"/>
 <pinref part="IC1" gate="G$1" pin="EN"/>
+<wire x1="48.26" y1="25.4" x2="55.88" y2="25.4" width="0.1524" layer="91"/>
 <wire x1="55.88" y1="25.4" x2="58.42" y2="25.4" width="0.1524" layer="91"/>
 <wire x1="58.42" y1="22.86" x2="55.88" y2="22.86" width="0.1524" layer="91"/>
@@
 <junction x="55.88" y="25.4"/>
 <junction x="40.64" y="25.4"/>
+<pinref part="C7" gate="G$1" pin="1"/>
+<wire x1="48.26" y1="22.86" x2="48.26" y2="25.4" width="0.1524" layer="91"/>
+<junction x="48.26" y="25.4"/>
 </segment>
 <segment>
@@
 <pinref part="C8" gate="G$1" pin="2"/>
 <pinref part="IC1" gate="G$1" pin="GND"/>
-<wire x1="40.64" y1="12.7" x2="68.58" y2="12.7" width="0.1524" layer="91"/>
+<wire x1="40.64" y1="12.7" x2="48.26" y2="12.7" width="0.1524" layer="91"/>
+<wire x1="48.26" y1="12.7" x2="68.58" y2="12.7" width="0.1524" layer="91"/>
 <wire x1="68.58" y1="12.7" x2="68.58" y2="17.78" width="0.1524" layer="91"/>
 <pinref part="C4" gate="G$1" pin="2"/>
@@
 <junction x="81.28" y="12.7"/>
 <junction x="40.64" y="12.7"/>
+<pinref part="C7" gate="G$1" pin="2"/>
+<wire x1="48.26" y1="15.24" x2="48.26" y2="12.7" width="0.1524" layer="91"/>
+<junction x="48.26" y="12.7"/>
 </segment>
 <segment>
@@
 </segment>
 <segment>
-<wire x1="40.64" y1="129.54" x2="40.64" y2="137.16" width="0.1524" layer="91"/>
-<wire x1="40.64" y1="129.54" x2="38.1" y2="124.46" width="0.1524" layer="91"/>
+<wire x1="38.1" y1="124.46" x2="38.1" y2="137.16" width="0.1524" layer="91"/>
 <pinref part="GND7" gate="1" pin="GND"/>
 <pinref part="U$1" gate="G$1" pin="GND"/>
@@
 <pinref part="GND14" gate="1" pin="GND"/>
 <pinref part="Q3" gate="G$1" pin="S"/>
-<wire x1="106.68" y1="116.84" x2="106.68" y2="119.38" width="0.1524" layer="91"/>
+<wire x1="106.68" y1="111.76" x2="106.68" y2="114.3" width="0.1524" layer="91"/>
+<pinref part="R8" gate="G$1" pin="1"/>
+<wire x1="106.68" y1="114.3" x2="106.68" y2="119.38" width="0.1524" layer="91"/>
+<wire x1="88.9" y1="116.84" x2="88.9" y2="114.3" width="0.1524" layer="91"/>
+<wire x1="88.9" y1="114.3" x2="106.68" y2="114.3" width="0.1524" layer="91"/>
+<junction x="106.68" y="114.3"/>
 </segment>
 <segment>
@@
 <net name="MOSI" class="0">
 <segment>
-<wire x1="53.34" y1="170.18" x2="53.34" y2="147.32" width="0.1524" layer="91"/>
-<wire x1="53.34" y1="147.32" x2="48.26" y2="147.32" width="0.1524" layer="91"/>
-<wire x1="48.26" y1="147.32" x2="48.26" y2="129.54" width="0.1524" layer="91"/>
-<wire x1="48.26" y1="129.54" x2="45.72" y2="124.46" width="0.1524" layer="91"/>
-<label x="53.34" y="154.94" size="1.778" layer="95" rot="MR90"/>
+<wire x1="45.72" y1="129.54" x2="45.72" y2="124.46" width="0.1524" layer="91"/>
+<label x="45.72" y="134.62" size="1.778" layer="95" rot="MR270"/>
 <pinref part="U$1" gate="G$1" pin="D11"/>
 </segment>
@@
 <net name="MISO" class="0">
 <segment>
-<wire x1="22.86" y1="147.32" x2="45.72" y2="147.32" width="0.1524" layer="91"/>
-<wire x1="45.72" y1="147.32" x2="45.72" y2="129.54" width="0.1524" layer="91"/>
-<wire x1="45.72" y1="129.54" x2="43.18" y2="124.46" width="0.1524" layer="91"/>
-<label x="35.56" y="147.32" size="1.778" layer="95" rot="MR0"/>
+<wire x1="43.18" y1="129.54" x2="43.18" y2="124.46" width="0.1524" layer="91"/>
+<label x="43.18" y="134.62" size="1.778" layer="95" rot="MR270"/>
 <pinref part="U$1" gate="G$1" pin="D12"/>
 </segment>
@@
 <net name="SCK" class="0">
 <segment>
-<wire x1="43.18" y1="129.54" x2="43.18" y2="149.86" width="0.1524" layer="91"/>
-<wire x1="43.18" y1="149.86" x2="25.4" y2="149.86" width="0.1524" layer="91"/>
-<wire x1="43.18" y1="129.54" x2="40.64" y2="124.46" width="0.1524" layer="91"/>
-<label x="35.56" y="149.86" size="1.778" layer="95" rot="MR0"/>
+<wire x1="40.64" y1="129.54" x2="40.64" y2="124.46" width="0.1524" layer="91"/>
+<label x="40.64" y="134.62" size="1.778" layer="95" rot="MR270"/>
 <pinref part="U$1" gate="G$1" pin="D13"/>
 </segment>
@@
 <net name="SD_CS" class="0">
 <segment>
-<wire x1="50.8" y1="129.54" x2="50.8" y2="144.78" width="0.1524" layer="91"/>
-<wire x1="50.8" y1="129.54" x2="48.26" y2="124.46" width="0.1524" layer="91"/>
-<wire x1="50.8" y1="144.78" x2="63.5" y2="144.78" width="0.1524" layer="91"/>
-<label x="60.96" y="144.78" size="1.778" layer="95" rot="MR0"/>
+<wire x1="48.26" y1="129.54" x2="48.26" y2="124.46" width="0.1524" layer="91"/>
+<label x="48.26" y="137.16" size="1.778" layer="95" rot="MR270"/>
 <pinref part="U$1" gate="G$1" pin="D10"/>
 </segment>
@@
 <wire x1="60.96" y1="129.54" x2="60.96" y2="124.46" width="0.1524" layer="91"/>
 <pinref part="U$1" gate="G$1" pin="D6"/>
-<wire x1="60.96" y1="129.54" x2="99.06" y2="129.54" width="0.1524" layer="91"/>
+<wire x1="60.96" y1="129.54" x2="88.9" y2="129.54" width="0.1524" layer="91"/>
+<wire x1="88.9" y1="129.54" x2="99.06" y2="129.54" width="0.1524" layer="91"/>
 <wire x1="99.06" y1="129.54" x2="99.06" y2="121.92" width="0.1524" layer="91"/>
 <pinref part="Q3" gate="G$1" pin="G"/>
 <wire x1="99.06" y1="121.92" x2="101.6" y2="121.92" width="0.1524" layer="91"/>
+<pinref part="R8" gate="G$1" pin="2"/>
+<wire x1="88.9" y1="127" x2="88.9" y2="129.54" width="0.1524" layer="91"/>
+<junction x="88.9" y="129.54"/>
 </segment>
 </net>
 <net name="N$108" class="0">
 <segment>
-<wire x1="38.1" y1="129.54" x2="35.56" y2="124.46" width="0.1524" layer="91"/>
+<wire x1="35.56" y1="129.54" x2="35.56" y2="124.46" width="0.1524" layer="91"/>
 <pinref part="U$1" gate="G$1" pin="AREF"/>
 </segment>
@@
 <net name="N$110" class="0">
 <segment>
-<wire x1="53.34" y1="129.54" x2="50.8" y2="124.46" width="0.1524" layer="91"/>
+<wire x1="50.8" y1="129.54" x2="50.8" y2="124.46" width="0.1524" layer="91"/>
 <pinref part="U$1" gate="G$1" pin="D9"/>
 </segment>

Commit message: Added accelerometer and barometer with associated level shifters. To be checked!
Parts:
- removed C1, C4: 10uF, rcl:C-USC0805
- added AP: (no value), pinhead:PINHD-1X3
- added C10: 4u7, rcl:C-USC0603
- added C11, C12, C13: 0.1uF, adafruit:C-USC0805
- added C14, C15: (no value), rcl:CPOL-USSMCB
- added C9: 220n, rcl:C-USC0603
- added IC5: BMP180, SparkFun-Sensors:BMP180
- added IC6: LSM9DS0, SparkFun-DigitalIC:LSM9DS0
- added Q4, Q5: MOSFET-NCHANNELBSS123LT1G, SparkFun-DiscreteSemi:MOSFET-NCHANNELBSS123LT1G
- added R10, R11, R12, R9: 10k, rcl:R-US_R0805
- added R13, R14: 4k7, adafruit:R-US_R0805
- R1, R2: value 2.2K -> 10k
Connections:
- removed net I2C_SCL: IC4.SCL, R1.2, SENSOR.3, U$1.A5
- removed net I2C_SDA: IC4.SDA, R2.2, SENSOR.4, U$1.A4
- removed net N$108: U$1.AREF
- removed net N$110: U$1.D9
- new net DHT22: SENSOR.5, U$1.A3
- new net I2C_3V3_SCL: IC5.SCL, IC6.SCL, Q4.S, R13.2
- new net I2C_3V3_SDA: IC5.SDA, IC6.SDA, Q5.S, R14.2
- new net I2C_5V_SCL: AP.1, IC4.SCL, Q4.D, R1.2, SENSOR.3, U$1.A5
- new net I2C_5V_SDA: AP.2, IC4.SDA, Q5.D, R2.2, SENSOR.4, U$1.A4
- new net N$11: IC6.SDO(XM), R9.1
- new net N$13: IC6.CS(XM), R10.1
- new net N$14: IC6.SDO(G), R11.1
- new net N$15: IC6.CS(G), R12.1
- new net N$16: C10.1, IC6.C1
- new net N$17: C9.1, IC6.SETC
- new net N$18: C9.2, IC6.SETP
- net +3V3: now also C11.1, C12.1, C15.+, IC5.VDD, IC5.VDDIO, IC6.VDD, IC6.VDD_IO, Q4.G, Q5.G, R10.2, R11.2, R12.2, R13.1, R14.1, R9.2; no longer C4.1, R7.1
- net +5V: now also C13.1, C14.+, R7.1; no longer C1.1, SENSOR.5
- net GND: now also AP.3, C10.2, C11.2, C12.2, C13.2, C14.-, C15.-, IC5.GND, IC6.GND; no longer C1.2, C4.2
Other:
- note added: "5V pull ups 10k as UV board has integral 10k pullups"
- note added: "Accelerometer"
- note added: "Barometer"
- note added: "I2C level shifter"
- note added: "f = 1.44 / (R4*C6) mark/space by R4"
- note removed: "f = 1.44 / (R4*C6)"
- moved on the sheet: C2, C7, C8, IC3A, IC3B, IC3C, LED3, LED4, R1, R2, R5, R6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

Commit message: Added DHT22 pullup and tidied up
Parts:
- added R15: 4k7, rcl:R-EU_R0805
Connections:
- net +5V: now also R15.2
- net DHT22: now also R15.1
Other:
- note added: "3M 2908-05WB-MG"
- note added: "Flash timer"
- note added: "RTC"
- moved on the sheet: AP, BAT, C10, C11, C12, C13, C14, C15, C2, C3, C5, C6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

Commit message: Final check, added BOM as .csv
Parts:
- removed LED4: red, adafruit:LEDCHIPLED_0805
- added LED1: (no value), led:LEDCHIPLED_0805
- C14, C15: value (none) -> 47u
- IC1: value LD6806 -> (none); device AWJLEagleLib:LD6806 -> AWJLEagleLib:MCP1700TT
- R6: value (none) -> 1k
Connections:
- net +5V: no longer IC1.EN
- net GND: now also LED1.C; no longer LED4.C
- net N$6: now also LED1.A; no longer LED4.A
Changed lines of the file:
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@@
 <part name="GND9" library="supply1" deviceset="GND" device=""/>
 <part name="+3V2" library="supply1" deviceset="+3V3" device=""/>
-<part name="R6" library="rcl" deviceset="R-EU_" device="R0805"/>
+<part name="R6" library="rcl" deviceset="R-EU_" device="R0805" value="1k"/>
 <part name="LED3" library="led" deviceset="LED" device="CHIPLED_0805"/>
 <part name="GND10" library="supply1" deviceset="GND" device=""/>
@@
 <part name="GND3" library="supply1" deviceset="GND" device=""/>
 <part name="R7" library="adafruit" deviceset="R-US_" device="R0805" value="1k"/>
-<part name="LED4" library="adafruit" deviceset="LED" device="CHIPLED_0805" value="red"/>
 <part name="GND4" library="supply1" deviceset="GND" device=""/>
 <part name="FRAME2" library="frames" deviceset="A3L-LOC" device=""/>
 <part name="SENSOR" library="con-harting-ml" deviceset="ML6" device=""/>
-<part name="IC1" library="AWJLEagleLib" deviceset="LD6806" device=""/>
 <part name="C8" library="adafruit" deviceset="C-US" device="C0805" value="0.1uF"/>
 <part name="GND6" library="supply1" deviceset="GND" device=""/>
@@
 <part name="AP" library="pinhead" deviceset="PINHD-1X3" device=""/>
 <part name="GND18" library="supply1" deviceset="GND" device=""/>
-<part name="C15" library="rcl" deviceset="CPOL-US" device="SMCB"/>
-<part name="C14" library="rcl" deviceset="CPOL-US" device="SMCB"/>
+<part name="C15" library="rcl" deviceset="CPOL-US" device="SMCB" value="47u"/>
+<part name="C14" library="rcl" deviceset="CPOL-US" device="SMCB" value="47u"/>
 <part name="R15" library="rcl" deviceset="R-EU_" device="R0805" value="4k7"/>
+<part name="IC1" library="AWJLEagleLib" deviceset="MCP1700" device="TT"/>
+<part name="LED1" library="led" deviceset="LED" device="CHIPLED_0805"/>
 </parts>
 <sheets>
@@
 <instance part="GND3" gate="1" x="165.1" y="50.8" rot="MR0"/>
 <instance part="R7" gate="G$1" x="121.92" y="40.64" rot="R270"/>
-<instance part="LED4" gate="G$1" x="121.92" y="30.48"/>
 <instance part="GND4" gate="1" x="121.92" y="20.32"/>
 <instance part="FRAME2" gate="G$1" x="0" y="0"/>
 <instance part="SENSOR" gate="1" x="177.8" y="119.38"/>
-<instance part="IC1" gate="G$1" x="66.04" y="38.1"/>
 <instance part="C8" gate="G$1" x="35.56" y="33.02"/>
 <instance part="GND6" gate="1" x="58.42" y="213.36" rot="MR0"/>
@@
 <instance part="C14" gate="G$1" x="20.32" y="33.02"/>
 <instance part="R15" gate="G$1" x="177.8" y="132.08" rot="R180"/>
+<instance part="IC1" gate="G$1" x="66.04" y="38.1"/>
+<instance part="LED1" gate="G$1" x="121.92" y="30.48"/>
 </instances>
 <busses>
@@
 <junction x="27.94" y="38.1"/>
 <junction x="20.32" y="38.1"/>
-<pinref part="IC1" gate="G$1" pin="IN"/>
 <wire x1="35.56" y1="38.1" x2="43.18" y2="38.1" width="0.1524" layer="91"/>
 <pinref part="C8" gate="G$1" pin="1"/>
-<pinref part="IC1" gate="G$1" pin="EN"/>
 <wire x1="43.18" y1="38.1" x2="50.8" y2="38.1" width="0.1524" layer="91"/>
 <wire x1="50.8" y1="38.1" x2="55.88" y2="38.1" width="0.1524" layer="91"/>
 <wire x1="55.88" y1="38.1" x2="58.42" y2="38.1" width="0.1524" layer="91"/>
-<wire x1="58.42" y1="35.56" x2="55.88" y2="35.56" width="0.1524" layer="91"/>
-<wire x1="55.88" y1="35.56" x2="55.88" y2="38.1" width="0.1524" layer="91"/>
 <junction x="55.88" y="38.1"/>
 <junction x="35.56" y="38.1"/>
@@
 <junction x="50.8" y="38.1"/>
 <pinref part="C14" gate="G$1" pin="+"/>
+<pinref part="IC1" gate="G$1" pin="IN"/>
 </segment>
 <segment>
@@
 <junction x="27.94" y="25.4"/>
 <pinref part="C8" gate="G$1" pin="2"/>
-<pinref part="IC1" gate="G$1" pin="GND"/>
 <wire x1="35.56" y1="25.4" x2="43.18" y2="25.4" width="0.1524" layer="91"/>
 <wire x1="43.18" y1="25.4" x2="50.8" y2="25.4" width="0.1524" layer="91"/>
-<wire x1="50.8" y1="25.4" x2="68.58" y2="25.4" width="0.1524" layer="91"/>
-<wire x1="68.58" y1="25.4" x2="68.58" y2="30.48" width="0.1524" layer="91"/>
-<wire x1="68.58" y1="25.4" x2="81.28" y2="25.4" width="0.1524" layer="91"/>
+<wire x1="50.8" y1="25.4" x2="66.04" y2="25.4" width="0.1524" layer="91"/>
+<wire x1="66.04" y1="25.4" x2="81.28" y2="25.4" width="0.1524" layer="91"/>
 <wire x1="81.28" y1="25.4" x2="88.9" y2="25.4" width="0.1524" layer="91"/>
 <wire x1="88.9" y1="25.4" x2="96.52" y2="25.4" width="0.1524" layer="91"/>
@@
 <pinref part="C3" gate="G$1" pin="2"/>
 <wire x1="81.28" y1="27.94" x2="81.28" y2="25.4" width="0.1524" layer="91"/>
-<junction x="68.58" y="25.4"/>
 <junction x="81.28" y="25.4"/>
 <junction x="35.56" y="25.4"/>
@@
 <pinref part="C14" gate="G$1" pin="-"/>
 <pinref part="C15" gate="G$1" pin="-"/>
+<pinref part="IC1" gate="G$1" pin="GND"/>
+<wire x1="66.04" y1="30.48" x2="66.04" y2="25.4" width="0.1524" layer="91"/>
+<junction x="66.04" y="25.4"/>
 </segment>
 <segment>
@@
 <segment>
 <pinref part="GND4" gate="1" pin="GND"/>
-<pinref part="LED4" gate="G$1" pin="C"/>
 <wire x1="121.92" y1="22.86" x2="121.92" y2="25.4" width="0.1524" layer="91"/>
+<pinref part="LED1" gate="G$1" pin="C"/>
 </segment>
 <segment>
@@
 <pinref part="C3" gate="G$1" pin="1"/>
 <pinref part="+3V1" gate="G$1" pin="+3V3"/>
-<pinref part="IC1" gate="G$1" pin="OUT"/>
 <wire x1="73.66" y1="38.1" x2="81.28" y2="38.1" width="0.1524" layer="91"/>
 <wire x1="81.28" y1="35.56" x2="81.28" y2="38.1" width="0.1524" layer="91"/>
@@
 <junction x="96.52" y="38.1"/>
 <pinref part="C15" gate="G$1" pin="+"/>
+<pinref part="IC1" gate="G$1" pin="OUT"/>
 </segment>
 <segment>
@@
 <net name="N$6" class="0">
 <segment>
-<pinref part="LED4" gate="G$1" pin="A"/>
 <pinref part="R7" gate="G$1" pin="2"/>
 <wire x1="121.92" y1="33.02" x2="121.92" y2="35.56" width="0.1524" layer="91"/>
-</segment>
-</net>
+<pinref part="LED1" gate="G$1" pin="A"/>
+</segment>
+</net>
